Commit message: feat(piper_mujoco): add ros2_control admittance simulation with force injection
- Add admittance_controller + ft_sensor mock injection pipeline
- Add admittance_trajectory_bridge: FollowJointTrajectory → joint_references topic
- Add world_force_bridge: world-frame Wrench → ft_sensor_link injectors
- Add admittance_demo.py: demo script for trajectory + force injection
- Update URDF with ft_sensor_link and ros2_control interfaces
- Update ros2_controllers.yaml with admittance/injector controller configs
- Update launch file with ordered controller spawning and mock/physics modes
- Update CMakeLists.txt and package.xml for new scripts and dependencies

Co-Authored-By: Claude Sonnet 4.6 <noreply@anthropic.com>

File: src/piper_description/urdf/piper_description.xacro (robot description, xacro)
@@ -3,4 +3,5 @@
   name="piper"
   xmlns:xacro="http://ros.org/wiki/xacro">
+  <xacro:arg name="lock_joints_4_6" default="false"/>
 <!-- world -->
   <link name="world"/>
@@ -221,22 +222,20 @@
     </collision>
   </link>
-  <joint
-    name="joint4"
-    type="revolute">
-    <origin
-      xyz="-0.021984 -0.25075 0"
-      rpy="1.5708 0 0" />
-    <parent
-      link="link3" />
-    <child
-      link="link4" />
-    <axis
-      xyz="0 0 1" />
-    <limit
-      lower="-1.745"
-      upper="1.745"
-      effort="100"
-      velocity="5" />
-  </joint>
+  <xacro:if value="$(arg lock_joints_4_6)">
+    <joint name="joint4" type="fixed">
+      <origin xyz="-0.021984 -0.25075 0" rpy="1.5708 0 0" />
+      <parent link="link3" />
+      <child  link="link4" />
+    </joint>
+  </xacro:if>
+  <xacro:unless value="$(arg lock_joints_4_6)">
+    <joint name="joint4" type="revolute">
+      <origin xyz="-0.021984 -0.25075 0" rpy="1.5708 0 0" />
+      <parent link="link3" />
+      <child  link="link4" />
+      <axis   xyz="0 0 1" />
+      <limit  lower="-1.745" upper="1.745" effort="100" velocity="5" />
+    </joint>
+  </xacro:unless>
   <link
     name="link5">
@@ -319,22 +318,20 @@
     </collision>
   </link>
-  <joint
-    name="joint6"
-    type="revolute">
-    <origin
-      xyz="8.8259E-05 -0.091 0"
-      rpy="1.5708 0 0" />
-    <parent
-      link="link5" />
-    <child
-      link="link6" />
-    <axis
-      xyz="0 0 1" />
-    <limit
-      lower="-2.0944"
-      upper="2.0944"
-      effort="100"
-      velocity="3" />
-  </joint>
+  <xacro:if value="$(arg lock_joints_4_6)">
+    <joint name="joint6" type="fixed">
+      <origin xyz="8.8259E-05 -0.091 0" rpy="1.5708 0 0" />
+      <parent link="link5" />
+      <child  link="link6" />
+    </joint>
+  </xacro:if>
+  <xacro:unless value="$(arg lock_joints_4_6)">
+    <joint name="joint6" type="revolute">
+      <origin xyz="8.8259E-05 -0.091 0" rpy="1.5708 0 0" />
+      <parent link="link5" />
+      <child  link="link6" />
+      <axis   xyz="0 0 1" />
+      <limit  lower="-2.0944" upper="2.0944" effort="100" velocity="3" />
+    </joint>
+  </xacro:unless>
   <link
     name="gripper_base">
@@ -520,7 +517,11 @@
   <xacro:transmission_block tran_name="tran2" joint_name="joint2" motor_name="motor2"/>
   <xacro:transmission_block tran_name="tran3" joint_name="joint3" motor_name="motor3"/>
-  <xacro:transmission_block tran_name="tran4" joint_name="joint4" motor_name="motor4"/>
+  <xacro:unless value="$(arg lock_joints_4_6)">
+    <xacro:transmission_block tran_name="tran4" joint_name="joint4" motor_name="motor4"/>
+  </xacro:unless>
   <xacro:transmission_block tran_name="tran5" joint_name="joint5" motor_name="motor5"/>
-  <xacro:transmission_block tran_name="tran6" joint_name="joint6" motor_name="motor6"/>
+  <xacro:unless value="$(arg lock_joints_4_6)">
+    <xacro:transmission_block tran_name="tran6" joint_name="joint6" motor_name="motor6"/>
+  </xacro:unless>
   <xacro:transmission_block tran_name="tran7" joint_name="joint7" motor_name="motor7"/>
   <xacro:transmission_block tran_name="tran8" joint_name="joint8" motor_name="motor8"/>

File: src/piper_description/urdf/piper_description_mujoco.xacro (robot description, xacro)
@@ -22,4 +22,5 @@
 <robot name="piper" xmlns:xacro="http://ros.org/wiki/xacro">
   <xacro:arg name="use_mock_hardware" default="true"/>
+  <xacro:arg name="lock_joints_4_6" default="false"/>
   <!-- Include base robot description (links, joints, transmissions) -->
   <xacro:include filename="$(find piper_description)/urdf/piper_description.xacro"/>
@@ -53,4 +54,5 @@
         <!-- mock: no external package needed, joints mirror commands -->
         <plugin>mock_components/GenericSystem</plugin>
+        <param name="mock_sensor_commands">true</param>
       </xacro:if>
       <xacro:unless value="$(arg use_mock_hardware)">
@@ -90,4 +92,5 @@
       <state_interface name="velocity"/>
     </joint>
+    <xacro:unless value="$(arg lock_joints_4_6)">
     <joint name="joint4">
       <command_interface name="position">
@@ -100,4 +103,5 @@
       <state_interface name="velocity"/>
     </joint>
+    </xacro:unless>
     <joint name="joint5">
       <command_interface name="position">
@@ -110,4 +114,5 @@
       <state_interface name="velocity"/>
     </joint>
+    <xacro:unless value="$(arg lock_joints_4_6)">
     <joint name="joint6">
       <command_interface name="position">
@@ -120,4 +125,5 @@
       <state_interface name="velocity"/>
     </joint>
+    </xacro:unless>
     <!-- Gripper joints: position command only, no admittance control -->
     <joint name="joint7">
@@ -144,10 +150,22 @@
          to ros2_control state interfaces consumed by admittance_controller -->
     <sensor name="ft_sensor">
-      <state_interface name="force.x"/>
-      <state_interface name="force.y"/>
-      <state_interface name="force.z"/>
-      <state_interface name="torque.x"/>
-      <state_interface name="torque.y"/>
-      <state_interface name="torque.z"/>
+      <state_interface name="force.x">
+        <param name="initial_value">0.0</param>
+      </state_interface>
+      <state_interface name="force.y">
+        <param name="initial_value">0.0</param>
+      </state_interface>
+      <state_interface name="force.z">
+        <param name="initial_value">0.0</param>
+      </state_interface>
+      <state_interface name="torque.x">
+        <param name="initial_value">0.0</param>
+      </state_interface>
+      <state_interface name="torque.y">
+        <param name="initial_value">0.0</param>
+      </state_interface>
+      <state_interface name="torque.z">
+        <param name="initial_value">0.0</param>
+      </state_interface>
     </sensor>
   </ros2_control>
